File: kicad/projects/switch/switch.kicad_pcb (KiCad board)
At the start: 2 copper layers, 56 x 50 mm, 24 parts, among them J1 Motor_Driver, J2 BTS, J3 KartCon, J4 WS2812b, J5 2S Lipo, J6 Motor_Driver, Q1 AO4407A, Q2 AO4407A, SW1 SW_DP3T

Commit message: Schalter-Platinchen: J6 als Buchsenleiste fuer die Werks-Stiftleiste des BTS7960
Gleiche Bohrungen und Netze je Loch; durch die gespiegelte Nummerierung des
Buchsen-Footprints ist J6 jetzt 1:1 wie J1 belegt. Ueberlappende GND-Durch-
kontaktierung an Pad 1 entfernt. Bilder und Stueckliste neu exportiert.

Co-Authored-By: Claude Opus 5.5 <noreply@anthropic.com>
Parts:
- J6: footprint Connector_PinHeader_2.54mm:PinHeader_2x04_P2.54mm_Vertical -> Connector_PinSocket_2.54mm:PinSocket_2x04_P2.54mm_Vertical
- moved J6 2.54 mm to (90.5, 40.2)
Connections:
- J6 pad 1: +5V -> GND
- J6 pad 2: GND -> +5V
- J6 pad 7: /RPWM -> /LPWM
- J6 pad 8: /LPWM -> /RPWM
Routing:
- net GND: vias 87 -> 86
Changed lines of the file:
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@@
 		)
 	)
-	(footprint "Connector_PinHeader_2.54mm:PinHeader_2x04_P2.54mm_Vertical"
+	(footprint "Connector_PinSocket_2.54mm:PinSocket_2x04_P2.54mm_Vertical"
 		(layer "F.Cu")
-		(at 90.46 42.73 90)
-		(descr "Through hole straight pin header, 2x04, 2.54mm pitch, double rows")
-		(tags "Through hole pin header THT 2x04 2.54mm double row")
+		(at 90.46 40.19 90)
+		(descr "Through hole straight socket strip, 2x04, 2.54mm pitch, double rows (from Kicad 4.0.7), script generated")
+		(tags "Through hole socket strip THT 2x04 2.54mm double row")
 		(property "Reference" "J6"
-			(at 1.27 -2.38 90)
+			(at -1.27 -2.38 90)
 			(layer "F.SilkS")
 			(effects
@@
 		)
 		(property "Value" "Motor_Driver"
-			(at 1.27 10 90)
+			(at -1.27 10.39 90)
 			(layer "F.Fab")
 			(effects
@@
 			)
 		)
-		(property ki_fp_filters "Connector*:*_2x??_*")
 		(sheetname "/")
 		(sheetfile "switch.kicad_sch")
-		(units
-			(unit
-				(name "A")
-				(pins "1" "3" "5" "7" "2" "4" "6" "8")
-			)
-		)
 		(attr through_hole)
 		(duplicate_pad_numbers_are_jumpers no)
 		(fp_line
-			(start 3.92 -1.38)
-			(end 3.92 9)
+			(start 1.33 -1.33)
+			(end 1.33 0)
 			(stroke
 				(width 0.12)
@@
 		)
 		(fp_line
-			(start 1.27 -1.38)
-			(end 3.92 -1.38)
+			(start 0 -1.33)
+			(end 1.33 -1.33)
 			(stroke
 				(width 0.12)
@@
 		)
 		(fp_line
-			(start -1.38 -1.38)
-			(end 0 -1.38)
+			(start -1.27 -1.33)
+			(end -1.27 1.27)
 			(stroke
 				(width 0.12)
@@
 		)
 		(fp_line
-			(start -1.38 0)
-			(end -1.38 -1.38)
+			(start -3.87 -1.33)
+			(end -1.27 -1.33)
 			(stroke
 				(width 0.12)
@@
 		)
 		(fp_line
-			(start 1.27 1.27)
-			(end 1.27 -1.38)
+			(start -3.87 -1.33)
+			(end -3.87 8.95)
 			(stroke
 				(width 0.12)
@@
 		)
 		(fp_line
-			(start -1.38 1.27)
-			(end 1.27 1.27)
+			(start 1.33 1.27)
+			(end 1.33 8.95)
 			(stroke
 				(width 0.12)
@@
 		)
 		(fp_line
-			(start -1.38 1.27)
-			(end -1.38 9)
+			(start -1.27 1.27)
+			(end 1.33 1.27)
 			(stroke
 				(width 0.12)
@@
 		)
 		(fp_line
-			(start -1.38 9)
-			(end 3.92 9)
+			(start -3.87 8.95)
+			(end 1.33 8.95)
 			(stroke
 				(width 0.12)
@@
 			(layer "F.SilkS")
 		)
-		(fp_rect
-			(start -1.77 -1.77)
-			(end 4.32 9.39)
+		(fp_line
+			(start 1.77 -1.77)
+			(end 1.77 9.39)
+			(stroke
+				(width 0.05)
+				(type solid)
+			)
+			(layer "F.CrtYd")
+		)
+		(fp_line
+			(start -4.31 -1.77)
+			(end 1.77 -1.77)
+			(stroke
+				(width 0.05)
+				(type solid)
+			)
+			(layer "F.CrtYd")
+		)
+		(fp_line
+			(start 1.77 9.39)
+			(end -4.31 9.39)
 			(stroke
 				(width 0.05)
 				(type solid)
 			)
-			(fill no)
 			(layer "F.CrtYd")
 		)
 		(fp_line
-			(start 3.81 -1.27)
-			(end 3.81 8.89)
+			(start -4.31 9.39)
+			(end -4.31 -1.77)
+			(stroke
+				(width 0.05)
+				(type solid)
+			)
+			(layer "F.CrtYd")
+		)
+		(fp_line
+			(start 0.27 -1.27)
+			(end 1.27 -0.27)
 			(stroke
 				(width 0.1)
@@
 		)
 		(fp_line
-			(start 0 -1.27)
-			(end 3.81 -1.27)
+			(start -3.81 -1.27)
+			(end 0.27 -1.27)
 			(stroke
 				(width 0.1)
@@
 		)
 		(fp_line
-			(start -1.27 0)
-			(end 0 -1.27)
+			(start 1.27 -0.27)
+			(end 1.27 8.89)
 			(stroke
 				(width 0.1)
@@
 		)
 		(fp_line
-			(start 3.81 8.89)
-			(end -1.27 8.89)
+			(start 1.27 8.89)
+			(end -3.81 8.89)
 			(stroke
 				(width 0.1)
@@
 		)
 		(fp_line
-			(start -1.27 8.89)
-			(end -1.27 0)
+			(start -3.81 8.89)
+			(end -3.81 -1.27)
 			(stroke
 				(width 0.1)
@@
 		)
 		(fp_text user "${REFERENCE}"
-			(at 1.27 3.81 0)
+			(at -1.27 3.81 180)
 			(layer "F.Fab")
 			(effects
@@
 			(layers "*.Cu" "*.Mask")
 			(remove_unused_layers no)
-			(net "+5V")
-			(pinfunction "Pin_1_1")
-			(pintype "passive")
+			(net "GND")
 		)
 		(pad "2" thru_hole circle
-			(at 2.54 0 90)
+			(at -2.54 0 90)
 			(size 1.7 1.7)
 			(drill 1)
 			(layers "*.Cu" "*.Mask")
 			(remove_unused_layers no)
-			(net "GND")
-			(pinfunction "Pin_2_2")
-			(pintype "passive")
+			(net "+5V")
 		)
 		(pad "3" thru_hole circle
@@
 			(remove_unused_layers no)
 			(net "unconnected-(J6-Pin_3-Pad3)")
-			(pinfunction "Pin_3_3")
-			(pintype "no_connect")
 		)
 		(pad "4" thru_hole circle
-			(at 2.54 2.54 90)
+			(at -2.54 2.54 90)
 			(size 1.7 1.7)
 			(drill 1)
@@
 			(remove_unused_layers no)
 			(net "unconnected-(J6-Pin_4-Pad4)")
-			(pinfunction "Pin_4_4")
-			(pintype "no_connect")
 		)
 		(pad "5" thru_hole circle
@@
 			(remove_unused_layers no)
 			(net "+5V")
-			(pinfunction "Pin_5_5")
-			(pintype "passive")
 		)
 		(pad "6" thru_hole circle
-			(at 2.54 5.08 90)
+			(at -2.54 5.08 90)
 			(size 1.7 1.7)
 			(drill 1)
@@
 			(remove_unused_layers no)
 			(net "+5V")
-			(pinfunction "Pin_6_6")
-			(pintype "passive")
 		)
 		(pad "7" thru_hole circle
@@
 			(layers "*.Cu" "*.Mask")
 			(remove_unused_layers no)
-			(net "/RPWM")
-			(pinfunction "Pin_7_7")
-			(pintype "passive")
+			(net "/LPWM")
 		)
 		(pad "8" thru_hole circle
-			(at 2.54 7.62 90)
+			(at -2.54 7.62 90)
 			(size 1.7 1.7)
 			(drill 1)
 			(layers "*.Cu" "*.Mask")
 			(remove_unused_layers no)
-			(net "/LPWM")
-			(pinfunction "Pin_8_8")
-			(pintype "passive")
+			(net "/RPWM")
 		)
 		(embedded_fonts no)
-		(model "${KICAD10_3DMODEL_DIR}/Connector_PinHeader_2.54mm.3dshapes/PinHeader_2x04_P2.54mm_Vertical.step"
+		(model "${KICAD10_3DMODEL_DIR}/Connector_PinSocket_2.54mm.3dshapes/PinSocket_2x04_P2.54mm_Vertical.step"
 			(offset
 				(xyz 0 0 0)
@@
 	)
 	(via
-		(at 91.46 41.16)
-		(size 0.6)
-		(drill 0.3)
-		(layers "F.Cu" "B.Cu")
-		(free yes)
-		(net "GND")
-	)
-	(via
 		(at 99.4 62.4)
 		(size 0.6)
@@
 	)
 	(segment
+		(start 96.03 52.32)
+		(end 100.71 47.64)
+		(width 0.2)
+		(layer "F.Cu")
+		(net "/LPWM")
+	)
+	(segment
+		(start 100.71 42.82)
+		(end 98.08 40.19)
+		(width 0.2)
+		(layer "F.Cu")
+		(net "/LPWM")
+	)
+	(segment
+		(start 100.71 47.64)
+		(end 100.71 42.82)
+		(width 0.2)
+		(layer "F.Cu")
+		(net "/LPWM")
+	)
+	(segment
 		(start 98.36 43.01)
 		(end 98.08 42.73)
@@
 		(net "/RPWM")
 	)
-	(segment
-		(start 96.03 52.32)
-		(end 100.71 47.64)
-		(width 0.2)
-		(layer "F.Cu")
-		(net "/LPWM")
-	)
-	(segment
-		(start 100.71 42.82)
-		(end 98.08 40.19)
-		(width 0.2)
-		(layer "F.Cu")
-		(net "/LPWM")
-	)
-	(segment
-		(start 100.71 47.64)
-		(end 100.71 42.82)
-		(width 0.2)
-		(layer "F.Cu")
-		(net "/LPWM")
-	)
 	(zone
