File: kicad/projects/switch/switch.kicad_sch (KiCad schematic)
At the start: 18 parts, among them J1 Motor_Driver, J2 BTS, J3 KartCon, J4 WS2812b, J5 2S Lipo, J6 Motor_Driver, Q1 AO4407A, Q2 AO4407A, SW1 SW_DP3T

Commit message: Schalter-Platinchen: J6 als Buchsenleiste fuer die Werks-Stiftleiste des BTS7960
Gleiche Bohrungen und Netze je Loch; durch die gespiegelte Nummerierung des
Buchsen-Footprints ist J6 jetzt 1:1 wie J1 belegt. Ueberlappende GND-Durch-
kontaktierung an Pad 1 entfernt. Bilder und Stueckliste neu exportiert.

Co-Authored-By: Claude Opus 5.5 <noreply@anthropic.com>
Parts:
- J6: footprint Connector_PinHeader_2.54mm:PinHeader_2x04_P2.54mm_Vertical -> Connector_PinSocket_2.54mm:PinSocket_2x04_P2.54mm_Vertical
Connections:
- net +5V: now also J6.2 (Pin_2); no longer J6.1 (Pin_1)
- net GND: now also J6.1 (Pin_1); no longer J6.2 (Pin_2)
- net LPWM: now also J6.7 (Pin_7); no longer J6.8 (Pin_8)
- net RPWM: now also J6.8 (Pin_8); no longer J6.7 (Pin_7)
Changed lines of the file:
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@@
 		)
 	)
-	(label "LPWM"
+	(label "RPWM"
 		(at 173.99 92.71 0)
 		(effects
@@
 		)
 	)
-	(label "RPWM"
+	(label "LPWM"
 		(at 161.29 92.71 180)
 		(effects
@@
 	)
 	(symbol
-		(lib_id "power:GND")
+		(lib_id "power:+5V")
 		(at 173.99 85.09 90)
 		(unit 1)
@@
 			)
 		)
-		(property "Value" "GND"
+		(property "Value" "+5V"
 			(at 177.8 85.0899 90)
 			(show_name no)
@@
 	)
 	(symbol
-		(lib_id "power:+5V")
+		(lib_id "power:GND")
 		(at 161.29 85.09 90)
 		(unit 1)
@@
 			)
 		)
-		(property "Value" "+5V"
+		(property "Value" "GND"
 			(at 157.48 85.0899 90)
 			(show_name no)
@@
 			)
 		)
-		(property "Footprint" "Connector_PinHeader_2.54mm:PinHeader_2x04_P2.54mm_Vertical"
+		(property "Footprint" "Connector_PinSocket_2.54mm:PinSocket_2x04_P2.54mm_Vertical"
 			(at 166.37 87.63 0)
 			(hide yes)
